Commit message: modify position

File: orne_box_description/urdf/orne_box.urdf.xacro (robot description, xacro)
@@ -57,5 +57,5 @@
   </xacro:sensor_hokuyo>
   <xacro:sensor_hokuyo name="mirror_lidar" parent="base_link" size="0.05 0.05 0.05">
-    <origin xyz="0.4 0.0 0.3" rpy="${-PI} 0.175 0"/>
+    <origin xyz="0.43 0.0 0.34" rpy="0 0.314 0"/>
   </xacro:sensor_hokuyo>
 </robot>
