Commit message: add mirror lidar

File: orne_box_description/urdf/orne_box.gazebo.xacro (robot description, xacro)
@@ -188,3 +188,47 @@
       <material>Gazebo/Black</material>
     </gazebo>
+    <!-- mirror_lidar -->
+    <gazebo reference="mirror_lidar_link">
+      <sensor type="ray" name="mirror_lidar_sensor">
+        <pose>0 0 0 0 0 0</pose>
+        <visualize>$(arg laser_visual)</visualize>
+        <update_rate>10</update_rate>
+        <ray>
+          <scan>
+            <horizontal>
+              <samples>341</samples>
+              <resolution>1</resolution>
+              <min_angle>${-PI/180*60}</min_angle>
+              <max_angle>${ PI/180*60}</max_angle>
+            </horizontal>
+            <vertical>
+              <samples>1</samples>
+              <resolution>1</resolution>
+            </vertical>
+          </scan>
+          <range>
+            <min>0.10</min>
+            <max>5.6</max>
+            <resolution>0.001</resolution>
+          </range>
+          <noise>
+            <type>gaussian</type>
+            <!-- Noise parameters based on published spec for Hokuyo laser
+                 achieving "+-30mm" accuracy at range < 10m.  A mean of 0.0m and
+                 stddev of 0.01m will put 99.7% of samples within 0.03m of the true
+                 reading. -->
+            <mean>0.0</mean>
+            <stddev>0.01</stddev>
+          </noise>
+        </ray>
+        <plugin name="gazebo_ros_mirror_lidar_controller" filename="libgazebo_ros_ray_sensor.so">
+          <ros>
+            <remapping>~/out:=mirror_scan</remapping>
+          </ros>
+          <frame_name>mirror_lidar_link</frame_name>
+          <output_type>sensor_msgs/LaserScan</output_type>
+        </plugin>
+      </sensor>
+      <material>Gazebo/Black</material>
+    </gazebo>
 </robot>

File: orne_box_description/urdf/orne_box.urdf.xacro (robot description, xacro)
@@ -57,5 +57,5 @@
   </xacro:sensor_hokuyo>
   <xacro:sensor_hokuyo name="mirror_lidar" parent="base_link" size="0.05 0.05 0.05">
-    <origin xyz="-0.08 0.0 0.7" rpy="${-PI} 0.175 0"/>
+    <origin xyz="0.4 0.0 0.3" rpy="${-PI} 0.175 0"/>
   </xacro:sensor_hokuyo>
 </robot>

Commit message: add mirror

File: orne_box_description/urdf/orne_box.gazebo.xacro (robot description, xacro)
@@ -232,3 +232,91 @@
       <material>Gazebo/Black</material>
     </gazebo>
+    <!-- mirror_lidar -->
+    <gazebo reference="mirror_lidar_left_link">
+      <sensor type="ray" name="mirror_lidar_left_sensor">
+        <pose>0 0 0 0 0 0</pose>
+        <visualize>$(arg laser_visual)</visualize>
+        <update_rate>10</update_rate>
+        <ray>
+          <scan>
+            <horizontal>
+              <samples>341</samples>
+              <resolution>1</resolution>
+              <min_angle>${PI/180*90}</min_angle>
+              <max_angle>${PI/180*140}</max_angle>
+            </horizontal>
+            <vertical>
+              <samples>1</samples>
+              <resolution>1</resolution>
+            </vertical>
+          </scan>
+          <range>
+            <min>0.10</min>
+            <max>5.6</max>
+            <resolution>0.001</resolution>
+          </range>
+          <noise>
+            <type>gaussian</type>
+            <!-- Noise parameters based on published spec for Hokuyo laser
+                 achieving "+-30mm" accuracy at range < 10m.  A mean of 0.0m and
+                 stddev of 0.01m will put 99.7% of samples within 0.03m of the true
+                 reading. -->
+            <mean>0.0</mean>
+            <stddev>0.01</stddev>
+          </noise>
+        </ray>
+        <plugin name="gazebo_ros_mirror_lidar_left_controller" filename="libgazebo_ros_ray_sensor.so">
+          <ros>
+            <remapping>~/out:=mirror_left_scan</remapping>
+          </ros>
+          <frame_name>mirror_lidar_left_link</frame_name>
+          <output_type>sensor_msgs/LaserScan</output_type>
+        </plugin>
+      </sensor>
+      <material>Gazebo/Black</material>
+    </gazebo>
+    <!-- mirror_lidar -->
+    <gazebo reference="mirror_lidar_right_link">
+      <sensor type="ray" name="mirror_lidar_right_sensor">
+        <pose>0 0 0 0 0 0</pose>
+        <visualize>$(arg laser_visual)</visualize>
+        <update_rate>10</update_rate>
+        <ray>
+          <scan>
+            <horizontal>
+              <samples>341</samples>
+              <resolution>1</resolution>
+              <min_angle>${-PI/180*140}</min_angle>
+              <max_angle>${-PI/180*90}</max_angle>
+            </horizontal>
+            <vertical>
+              <samples>1</samples>
+              <resolution>1</resolution>
+            </vertical>
+          </scan>
+          <range>
+            <min>0.10</min>
+            <max>5.6</max>
+            <resolution>0.001</resolution>
+          </range>
+          <noise>
+            <type>gaussian</type>
+            <!-- Noise parameters based on published spec for Hokuyo laser
+                 achieving "+-30mm" accuracy at range < 10m.  A mean of 0.0m and
+                 stddev of 0.01m will put 99.7% of samples within 0.03m of the true
+                 reading. -->
+            <mean>0.0</mean>
+            <stddev>0.01</stddev>
+          </noise>
+        </ray>
+        <plugin name="gazebo_ros_mirror_right_lidar_controller" filename="libgazebo_ros_ray_sensor.so">
+          <ros>
+            <remapping>~/out:=mirror_right_scan</remapping>
+          </ros>
+          <frame_name>mirror_lidar_right_link</frame_name>
+          <output_type>sensor_msgs/LaserScan</output_type>
+        </plugin>
+      </sensor>
+      <material>Gazebo/Black</material>
+    </gazebo>
 </robot>

File: orne_box_description/urdf/orne_box.urdf.xacro (robot description, xacro)
@@ -59,3 +59,11 @@
     <origin xyz="0.43 0.0 0.34" rpy="0 0.314 0"/>
   </xacro:sensor_hokuyo>
+  <xacro:property name="left_angle" value="70"/>
+  <xacro:sensor_hokuyo name="mirror_lidar_left" parent="mirror_lidar_link" size="0.05 0.05 0.05">
+    <origin xyz="0.0 ${0.21*(1.0-cos(radians(left_angle)))} ${0.21*sin(radians(left_angle))}" rpy="${-radians(left_angle)} 0 0"/>
+  </xacro:sensor_hokuyo>
+  <xacro:property name="right_angle" value="70"/>
+  <xacro:sensor_hokuyo name="mirror_lidar_right" parent="mirror_lidar_link" size="0.05 0.05 0.05">
+    <origin xyz="0.0 ${-0.21*(1.0-cos(radians(right_angle)))} ${0.21*sin(radians(right_angle))}" rpy="${radians(right_angle)} 0 0"/>
+  </xacro:sensor_hokuyo>
 </robot>
